File: hardware/v0.2/spi_fiend.kicad_pcb (KiCad board)
At the start: 4 copper layers, 34.8 x 18 mm, 25 parts, among them J1 USB_C_Receptacle_USB2.0, J2 CONN_01X04, J3 CONN_01X07, J4 PROG HEADER, J5 CONN_01X05, SW1 SW_Push, SW2 SW_Push, U1 STM32F042G6U6, U2 DRTR5V0U4S, U3 XC6222B331MR-G

Commit message: Revert "P&R almost done."
This reverts commit 97a49ac74aeb3e6297260b20c9d5898586bb1314.
Parts:
- moved J3 46.7 mm to (119.1, 88.5)
- moved J5 42.9 mm to (123.7, 88.5), turned to 0 degrees
- moved R7 37.2 mm to (154.0, 87.1), turned to 0 degrees
- moved R1 32.5 mm to (146.0, 95.6), turned to 0 degrees
- moved C3 31.2 mm to (154.0, 89.1), turned to 0 degrees
- moved J4 29.9 mm to (142.6, 90.4)
- moved R6 27.3 mm to (148.9, 91.6), turned to 0 degrees
- moved SW2 26.9 mm to (141.1, 97.0), turned to 0 degrees
- moved J1 26.1 mm to (131.9, 91.9), turned to 0 degrees
- moved R2 26.1 mm to (143.0, 100.3), turned to 0 degrees
- moved U3 26.0 mm to (150.0, 88.4)
- moved J2 25.7 mm to (128.4, 98.9), turned to 0 degrees
- moved D3 25.3 mm to (139.5, 100.6), turned to 0 degrees
- moved SW1 25.3 mm to (134.1, 99.0), turned to 0 degrees
- moved C4 22.8 mm to (148.8, 93.6), turned to 0 degrees
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Connections:
- C2 pad 1: +3.3V -> +3V3
- C3 pad 1: +3.3V -> +3V3
- J5 pad 1: +3.3V -> +3V3
- R1 pad 1: +3.3V -> +3V3
- SW2 pad 1: +3.3V -> +3V3
- U1 pad 17: +3.3V -> +3V3
- U1 pad 18: +3.3V -> +3V3
- U1 pad 5: +3.3V -> +3V3
Routing:
- net /NRST: track 30.0 -> 0.00 mm, vias 2 -> 0
- net /SO: track 27.4 -> 0.00 mm, vias 1 -> 0
- net /SI: track 26.9 -> 0.00 mm, vias 1 -> 0
- net /SPI_CS: track 24.5 -> 0.00 mm
- net GND: track 22.1 -> 0.00 mm, vias 17 -> 0
- net /CDONE: track 21.8 -> 0.00 mm, vias 2 -> 0
- net /VUSB: track 21.5 -> 0.00 mm, vias 3 -> 0
- net /CRESET: track 20.1 -> 0.00 mm
- net /SPI_SCLK: track 19.7 -> 0.00 mm, vias 1 -> 0
- net Net-(J1-PadS1): track 18.8 -> 0.00 mm
- net /SWDIO: track 17.4 -> 0.00 mm
- net +3.3V: track 15.3 -> 0.00 mm, vias 6 -> 0
- net /LED0: track 13.2 -> 0.00 mm, vias 2 -> 0
- net /LED1: track 12.8 -> 0.00 mm, vias 2 -> 0
- net /USB_DM: track 12.2 -> 0.00 mm
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- removed copper zone on In2.Cu, net +3.3V
- removed copper zone on In1.Cu, net GND
Other:
- board outline removed
- copper layers 4 -> 2
- rule pad_to_mask_clearance: 0.051 -> 0
- board text removed: "BOOT"
- board text removed: "DIR"
- board text removed: "ERR"
- board text removed: "PWR"
- board text removed: "RST"
