File: hardware/v0.2/spi_fiend.kicad_pcb (KiCad board)
At the start: 2 copper layers, 25 parts, among them J1 USB_C_Receptacle_USB2.0, J2 CONN_01X04, J3 CONN_01X07, J4 PROG HEADER, J5 CONN_01X05, SW1 SW_Push, SW2 SW_Push, U1 STM32F042G6U6, U2 DRTR5V0U4S, U3 XC6222B331MR-G

Commit message: P&R almost done.
Parts:
- moved J3 46.7 mm to (160.4, 110.4)
- moved J5 42.9 mm to (146.6, 124.8), turned to 90 degrees
- moved R7 37.2 mm to (136.8, 120.1), turned to 180 degrees
- moved R1 32.5 mm to (135.0, 126.2), turned to 180 degrees
- moved C3 31.2 mm to (140.4, 117.2), turned to 180 degrees
- moved J4 29.9 mm to (153.7, 118.1)
- moved R6 27.3 mm to (136.8, 116.1), turned to 180 degrees
- moved SW2 26.9 mm to (142.6, 123.8), turned to 90 degrees
- moved J1 26.1 mm to (129.9, 118.0), turned to -90 degrees
- moved R2 26.1 mm to (135.0, 125.1), turned to 180 degrees
- moved U3 26.0 mm to (137.5, 111.1)
- moved J2 25.7 mm to (151.1, 111.0), turned to 90 degrees
- moved D3 25.3 mm to (133.0, 125.0), turned to 90 degrees
- moved SW1 25.3 mm to (138.7, 123.8), turned to 90 degrees
- moved C4 22.8 mm to (134.3, 111.2), turned to -90 degrees
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Connections:
- C2 pad 1: +3V3 -> +3.3V
- C3 pad 1: +3V3 -> +3.3V
- J5 pad 1: +3V3 -> +3.3V
- R1 pad 1: +3V3 -> +3.3V
- SW2 pad 1: +3V3 -> +3.3V
- U1 pad 17: +3V3 -> +3.3V
- U1 pad 18: +3V3 -> +3.3V
- U1 pad 5: +3V3 -> +3.3V
Routing:
- net /NRST: track 0.00 -> 30.0 mm, vias 0 -> 2
- net /SO: track 0.00 -> 27.4 mm, vias 0 -> 1
- net /SI: track 0.00 -> 26.9 mm, vias 0 -> 1
- net /SPI_CS: track 0.00 -> 24.5 mm
- net GND: track 0.00 -> 22.1 mm, vias 0 -> 17
- net /CDONE: track 0.00 -> 21.8 mm, vias 0 -> 2
- net /VUSB: track 0.00 -> 21.5 mm, vias 0 -> 3
- net /CRESET: track 0.00 -> 20.1 mm
- net /SPI_SCLK: track 0.00 -> 19.7 mm, vias 0 -> 1
- net Net-(J1-PadS1): track 0.00 -> 18.8 mm
- net /SWDIO: track 0.00 -> 17.4 mm
- net +3.3V: track 0.00 -> 15.3 mm, vias 0 -> 6
- net /LED0: track 0.00 -> 13.2 mm, vias 0 -> 2
- net /LED1: track 0.00 -> 12.8 mm, vias 0 -> 2
- net /USB_DM: track 0.00 -> 12.2 mm
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- added copper zone on In2.Cu, net +3.3V
- added copper zone on In1.Cu, net GND
Other:
- board outline added: 34.8 x 18 mm
- copper layers 2 -> 4
- rule pad_to_mask_clearance: 0 -> 0.051
- board text added: "BOOT"
- board text added: "DIR"
- board text added: "ERR"
- board text added: "PWR"
- board text added: "RST"

Commit message: Done
Parts:
- added R4: 1k, Resistor_SMD:R_0402_1005Metric, F.Cu at (147.8, 113.2)
- added R5: 1k, Resistor_SMD:R_0402_1005Metric, F.Cu at (144.9, 113.2)
- added Ref**: Val**, emeb_library:avatar_small, B.Cu at (142.2, 115.8)
- moved D1 0.13 mm to (128.5, 125.0)
- moved D2 0.13 mm to (130.8, 125.0)
- moved D3 0.13 mm to (133.1, 125.0)
- renumbered R4 to R6, R5 to R7, R6 to R8, R7 to R9
Connections:
- J4 pad 10: /SPARE10 -> /RX
- J4 pad 8: +3.3V -> /Vt
- J4 pad 9: /SPARE9 -> /TX
- U1 pad 6: unconnected-(U1-Pad6) -> Net-(U1-Pad6)
Routing:
- net /Vt: track 0.00 -> 16.5 mm, vias 0 -> 2
- net /RX: track 11.6 -> 23.8 mm, vias 1 -> 2
- net /TX: track 8.06 -> 19.9 mm, vias 1 -> 2
- net Net-(U1-Pad6): track 0.00 -> 7.50 mm, vias 0 -> 2
- net GND: track 22.1 -> 25.5 mm
- net +3.3V: track 15.3 -> 13.7 mm, vias 6 -> 5
Other:
- board text added: "CDN"
- board text added: "CLK"
- board text added: "CRS"
- board text added: "CS"
- board text added: "GND"
- board text added: "NRST"
- board text added: "RX"
- board text added: "SI"
- board text added: "SO"
- board text added: "SPI Fiend V0.2"
- board text added: "SPI Fiend V0.2 (c) 2022 E. Brombaugh"
- board text added: "SWCLK"
- board text added: "SWDIO"
- board text added: "TX"
- board text added: "VDD"
- board text added: "VT"
