File: hardware/v0.2/spi_fiend.kicad_sch (KiCad schematic)
At the start: 25 parts, among them J1 USB_C_Receptacle_USB2.0, J2 CONN_01X04, J3 CONN_01X07, J4 PROG HEADER, J5 CONN_01X05, SW1 SW_Push, SW2 SW_Push, U1 STM32F042G6U6, U2 DRTR5V0U4S, U3 XC6222B331MR-G

Commit message: Done
Parts:
- added R4, R5: 1k, Resistor_SMD:R_0402_1005Metric, symbol Device:R
- renumbered R4 to R6, R5 to R7, R6 to R8, R7 to R9
Connections:
- net SPARE10 is gone; now on net RX: J4.10 (Pin_10)
- net SPARE9 is gone; now on net TX: J4.9 (Pin_9)
- net +3.3V: no longer J4.8 (Pin_8)
- net GND: now also R5.1
- net at U1.6 (PA0): now also R4.2, R5.2
- new net Vt: J4.8 (Pin_8), R4.1
- no-connect marks 10 -> 9
Other:
- note added: "SPARE10 [FPGA TX]"
- note added: "SPARE9 [FPGA RX]"
- note removed: "RX"
- note removed: "TX"
